File: hardware/pullometer.kicad_pcb (KiCad board)
At the start: 2 copper layers, 96.5 x 45.7 mm, 49 parts, among them P1 BATTERY, P2 SG1, P3 SG2, P4 DEBUG, P5 SG3, Q1 MMBT4403, Q2 TMS2302CX, SW1 RESET, SW2 POWER, U1 nRF24L01, U2 LTC3621, U3 MCP1702, U4 MKL05Z32VLC4, U5 HX711, U6 GY-85, Y1 32.768kHz

Commit message: Production hardware
Signed-off-by: Paul Brook <paul@nowt.org>
Parts:
- added G***: OSHW_LOGO, Parts:OSHW_LOGO, F.Cu at (184.2, 101.0)
- added R1: 1M, Parts:R_0805_HandSoldering_V, F.Cu at (181.6, 125.7)
- added R2: 0R, Parts:R_0805_HandSoldering_V, F.Cu at (171.4, 114.3)
- C1, C3: value 22uF -> 22u; footprint Capacitors_SMD:C_0805_HandSoldering -> Parts:C_0805_HandSoldering_V
- C10, C12, C13, C14, C6, C8: value 0.1uF -> 0.1u; footprint Capacitors_SMD:C_0805_HandSoldering -> Parts:C_0805_HandSoldering_V
- C11, C7, C9: value 10uF -> 10u; footprint Capacitors_SMD:C_0805_HandSoldering -> Parts:C_0805_HandSoldering_V
- C2, C4, C5: value 1uF -> 1u; footprint Capacitors_SMD:C_0805_HandSoldering -> Parts:C_0805_HandSoldering_V
- D1: footprint Diodes_ThroughHole:Diode_DO-41_SOD81_Horizontal_RM10 -> Discret:DO-41
- P1, P2, P3: footprint Pin_Headers:Pin_Header_Straight_1x02 -> Parts:JST-XH-2
- P5: footprint Pin_Headers:Pin_Header_Straight_1x04 -> Parts:JST-XH-4
- R10, R11, R12, R13, R14, R15, R16, R17, R4, R5, R6, R7, R8, R9: footprint Resistors_SMD:R_0805_HandSoldering -> Parts:R_0805_HandSoldering_V
- SW2: footprint Buttons_Switches_ThroughHole:SW_DIP_x1_Slide -> Buttons_Switches_ThroughHole:SW_Micro_SPST
- moved R4 15.9 mm to (181.6, 130.8), turned to 270 degrees
- moved P5 13.3 mm to (120.7, 109.2), turned to 270 degrees
- moved P3 12.8 mm to (120.7, 132.1), turned to 270 degrees
- moved P2 12.8 mm to (120.7, 121.9), turned to 270 degrees
- moved R16 11.7 mm to (139.7, 132.1), turned to 270 degrees
- moved R15 10.9 mm to (137.2, 132.1), turned to 270 degrees
- moved JP1 10.2 mm to (125.7, 119.4)
- moved SW1 10.2 mm to (128.3, 108.0)
- moved R9 10.2 mm to (130.8, 119.4)
- moved JP2 10.2 mm to (125.7, 130.8)
- moved R12 10.2 mm to (130.8, 130.8)
- moved C5 8.98 mm to (163.8, 128.3)
- moved R13 8.98 mm to (129.5, 127.0), turned to 270 degrees
- moved U3 8.89 mm to (163.8, 132.1)
- moved R10 8.89 mm to (129.5, 115.6), turned to 270 degrees
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Connections:
- U4 pad 12: /RUN -> /S_RUN
- U5 pad 10: Net-(C13-Pad1) -> Net-(C13-Pad2)
- U5 pad 9: Net-(C13-Pad2) -> Net-(C13-Pad1)
Routing:
- net +3V3: track 156.7 -> 139.3 mm, vias 2 -> 1
- net GND: track 74.1 -> 59.2 mm, vias 9 -> 10
- net /IN-: track 41.4 -> 29.5 mm, vias 0 -> 1
- net /IN+: track 50.1 -> 39.7 mm, vias 0 -> 1
- net /RUN: track 34.3 -> 25.1 mm
- net /Vbat: track 59.7 -> 50.9 mm
- net /BAT_EN: track 33.7 -> 26.3 mm
- net /E+: track 77.2 -> 69.8 mm, vias 3 -> 0
- net /HX_DATA: track 14.3 -> 7.45 mm
- net Net-(C13-Pad1): track 23.7 -> 17.0 mm
- net /S_RUN: track 0.00 -> 6.57 mm
- net /SWD_RESET: track 60.0 -> 54.7 mm
- net /HX_RATE: track 12.7 -> 7.51 mm
- net /UART_RX: track 44.3 -> 39.4 mm
- net /MOSI: track 16.6 -> 12.3 mm
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Other:
- board size 96.5 x 45.7 mm -> 77.5 x 45.7 mm
- board text added: "+"
- board text added: "-"
- board text added: "150"
- board text added: "300"
- board text added: "3v3"
- board text added: "CLK"
- board text added: "DIO"
- board text added: "E"
- board text added: "G"
- board text added: "GND"
- board text added: "Pull-o-meter"
- board text added: "RST"
- board text added: "RX"
- board text added: "TX"
- board text added: "©Paul Brook"
